File: V1/ESP-pwm_8ch-V1.kicad_pcb (KiCad board)
At the start: 2 copper layers, 123 x 67.8 mm, 46 parts, among them J1 12VDC, J2 CH1/2, J3 CH3/4, J4 CH5/6, J5 CH7/8, Q1 IRLB8721PBF, Q2 IRLB8721PBF, Q3 IRLB8721PBF, Q4 IRLB8721PBF, Q5 IRLB8721PBF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

Commit message: work in progress
Parts:
- added REF**: OSHW-Logo2_14.6x12mm_SilkScreen, Symbol:OSHW-Logo2_14.6x12mm_SilkScreen, F.Cu at (95.2, 74.9)
- moved D2 3.17 mm to (72.5, 67.9)
- moved D3 3.17 mm to (72.5, 75.6)
- moved D4 3.17 mm to (72.5, 71.8)
- moved REF** 1.27 mm to (95.2, 125.7)
Routing:
- net Net-(D4-Pad2): track 22.8 -> 21.5 mm
- net Net-(D3-Pad2): track 18.0 -> 16.7 mm
- net Net-(D2-Pad2): track 27.7 -> 26.4 mm
- net GNDREF: track 471.2 -> 469.9 mm
Other:
- board size 123 x 67.8 mm -> 113 x 67.8 mm
- board text added: "DESIGNED BY TALES MASCHIO 2022"
- board text added: "SUPORTES PCI METALTEX SP7 1x pé macho 9 mm 1x pé fêmea 9 mm 1x espaçador 20 mm 1x espaçador 30 mm 1x espaçador 45 mm Comprimento total 113 mm Largura da placa 67,8 mm"
- board text removed: "SUPORTES PCI METALTEX SP7 1x pé macho 9 mm 1x pé fêmea 9 mm 4x espaçador 20 mm 1x espaçador 45 mm Comprimento total 143 mm Largura da placa 67,8 mm"

Commit message: wip
Parts:
- removed the REF** at (95.2, 125.7)
- added G***: LOGO, Tales:TMaschio_20mm, F.Cu at (95.2, 82.5)
- moved REF** 2.54 mm to (95.2, 72.4)
Routing:
- net GNDREF: track 469.9 -> 465.4 mm
Other:
- board text added: "MAX LOAD 5A/CHANNEL"
- board text removed: "DESIGNED BY TALES MASCHIO 2022"
- board text removed: "MAX LOAD 5 A PER CHANNEL"
