File: V1/ESP-pwm_8ch-V1.kicad_sch (KiCad schematic)
At the start: 47 parts, among them J1 12VDC, J2 CH1/2, J3 CH3/4, J4 CH5/6, J5 CH7/8, Q1 IRLB8721PBF, Q2 IRLB8721PBF, Q3 IRLB8721PBF, Q4 IRLB8721PBF, Q5 IRLB8721PBF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

Commit message: PCB tweaks
Other:
- note added: "ESP8266 D6/GPIO12 (5) -> OUT 1 D5/GPIO14 (4) -> OUT 2 D2/GPIO4 (13) -> OUT 3 D1/GPIO5 (14) -> OUT 4 ESP32 GPIO33 (16) -> OUT 1 GPIO32 (15) -> OUT 2 GPIO16 (14) -> OUT 3 GPIO15 (13) -> OUT 4 GPIO13 (11) -> OUT 5 GPIO14 (12) -> OUT 6 GPIO5 (10) -> OUT 7 GPIO4 (9) -> OUT 8"
- note removed: "ESP32 GPIO33 (13) -> OUT 1 GPIO32 (14) -> OUT 2 GPIO16 (15) -> OUT 3 GPIO15 (16) -> OUT 4 GPIO13 (11) -> OUT 5 GPIO14 (12) -> OUT 6 GPIO4 (09) -> OUT 7 GPIO5 (10) -> OUT 8"
- note removed: "ESP8266 GPIO33 (13) -> OUT 1 GPIO32 (14) -> OUT 2 GPIO16 (15) -> OUT 3 GPIO15 (16) -> OUT 4"
Changed lines of the file:
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@@
     (stroke (width 0) (type default) (color 0 0 0 0))
   )
-  (wire (pts (xy 93.98 234.95) (xy 196.85 234.95))
+  (wire (pts (xy 105.41 234.95) (xy 196.85 234.95))
     (stroke (width 0) (type default) (color 0 0 0 0))
   )
@@
     (stroke (width 0) (type default) (color 0 0 0 0))
   )
-  (wire (pts (xy 99.06 203.2) (xy 99.06 240.03))
+  (wire (pts (xy 110.49 203.2) (xy 110.49 240.03))
     (stroke (width 0) (type default) (color 0 0 0 0))
   )
@@
     (stroke (width 0) (type default) (color 0 0 0 0))
   )
-  (wire (pts (xy 99.06 240.03) (xy 199.39 240.03))
+  (wire (pts (xy 110.49 240.03) (xy 199.39 240.03))
     (stroke (width 0) (type default) (color 0 0 0 0))
   )
@@
     (stroke (width 0) (type default) (color 0 0 0 0))
   )
-  (wire (pts (xy 120.65 200.66) (xy 93.98 200.66))
+  (wire (pts (xy 120.65 200.66) (xy 105.41 200.66))
     (stroke (width 0) (type default) (color 0 0 0 0))
   )
@@
     (stroke (width 0) (type default) (color 0 0 0 0))
   )
-  (wire (pts (xy 120.65 203.2) (xy 99.06 203.2))
+  (wire (pts (xy 120.65 203.2) (xy 110.49 203.2))
     (stroke (width 0) (type default) (color 0 0 0 0))
   )
@@
     (stroke (width 0) (type default) (color 0 0 0 0))
   )
-  (wire (pts (xy 93.98 200.66) (xy 93.98 234.95))
+  (wire (pts (xy 105.41 200.66) (xy 105.41 234.95))
     (stroke (width 0) (type default) (color 0 0 0 0))
   )
@@
     (stroke (width 0) (type default) (color 0 0 0 0))
   )
-  (text "ESP8266\nGPIO33 (13) -> OUT 1\nGPIO32 (14) -> OUT 2\nGPIO16 (15) -> OUT 3\nGPIO15 (16) -> OUT 4\n"
-    (at 82.55 266.7 0)
-    (effects (font (size 2.5 2.5)) (justify left bottom))
-  )
-  (text "ESP32\nGPIO33 (13) -> OUT 1\nGPIO32 (14) -> OUT 2\nGPIO16 (15) -> OUT 3\nGPIO15 (16) -> OUT 4\nGPIO13 (11) -> OUT 5\nGPIO14 (12) -> OUT 6\nGPIO4  (09) -> OUT 7\nGPIO5  (10) -> OUT 8"
+  (text "ESP8266\nD6/GPIO12 (5) -> OUT 1\nD5/GPIO14 (4) -> OUT 2\nD2/GPIO4 (13) -> OUT 3\nD1/GPIO5 (14) -> OUT 4\n\nESP32\nGPIO33 (16) -> OUT 1\nGPIO32 (15) -> OUT 2\nGPIO16 (14) -> OUT 3\nGPIO15 (13) -> OUT 4\nGPIO13 (11) -> OUT 5\nGPIO14 (12) -> OUT 6\nGPIO5  (10) -> OUT 7\nGPIO4   (9) -> OUT 8"
     (at 20.32 278.13 0)
     (effects (font (size 2.5 2.5)) (justify left bottom))
@@
   (symbol (lib_id "Tales:Olimex_ESP32-POE") (at 139.7 198.12 0) (unit 1)
     (in_bom yes) (on_board yes)
-    (property "Reference" "U3" (id 0) (at 101.6 213.36 0)
+    (property "Reference" "U3" (id 0) (at 144.78 218.44 0)
       (effects (font (size 1.27 1.27)) (justify left))
     )
-    (property "Value" "Olimex_ESP32-POE" (id 1) (at 101.6 215.9 0)
+    (property "Value" "Olimex_ESP32-POE" (id 1) (at 144.78 220.98 0)
       (effects (font (size 1.27 1.27)) (justify left))
     )
@@
   (symbol (lib_id "power:+3.3V") (at 105.41 110.49 0) (unit 1)
     (in_bom yes) (on_board yes)
-    (property "Reference" "#PWR?" (id 0) (at 105.41 114.3 0)
+    (property "Reference" "#PWR010" (id 0) (at 105.41 114.3 0)
       (effects (font (size 1.27 1.27)) hide)
     )
@@
   )
   (symbol (lib_id "MCU_Module:WeMos_D1_mini") (at 139.7 133.35 0) (unit 1)
-    (in_bom yes) (on_board yes) (fields_autoplaced)
+    (in_bom yes) (on_board yes)
     (property "Reference" "U2" (id 0) (at 141.7194 153.67 0)
       (effects (font (size 1.27 1.27)) (justify left))
@@
       (reference "#PWR09") (unit 1) (value "GNDREF") (footprint "")
     )
+    (path "/23e77feb-3aa3-4dc3-be1d-77aac6d23b29"
+      (reference "#PWR010") (unit 1) (value "+3.3V") (footprint "")
+    )
     (path "/f751bbdd-6bc8-4a06-baee-162a4b18bd26"
       (reference "#PWR0101") (unit 1) (value "+VA") (footprint "")
@@
       (reference "#PWR0132") (unit 1) (value "+12VA") (footprint "")
     )
-    (path "/23e77feb-3aa3-4dc3-be1d-77aac6d23b29"
-      (reference "#PWR?") (unit 1) (value "+3.3V") (footprint "")
-    )
     (path "/00000000-0000-0000-0000-000062418b8f"
