File: V1/ESP-pwm-8ch-V1.kicad_pcb (KiCad board)
At the start: 2 copper layers, 113 x 67.8 mm, 49 parts, among them J1 12VDC, J2 CH1/2, J3 CH3/4, J4 CH5/6, J5 CH7/8, Q1 IRLB8721PBF, Q2 IRLB8721PBF, Q3 IRLB8721PBF, Q4 IRLB8721PBF, Q5 IRLB8721PBF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

Commit message: pcb tweaks
Other:
- board text added: "ESP-PWM-8CH-V1"
Changed lines of the file:
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@@
     (effects (font (size 1.8 1.8) (thickness 0.35)))
+  )
+  (gr_text "ESP-PWM-8CH-V1" (at 95.25 67.31) (layer "F.SilkS")
+    (effects (font (size 1.2 1.2) (thickness 0.2)))
   )
   (gr_text "12VDC 3/4" (at 149.86 129.54) (layer "F.SilkS")

Commit message: Separated driver power lines from loads
Parts:
- turned D3 to 0 degrees
Connections:
- C10 pad 1: +VD -> +12VA
- C11 pad 1: +VD -> +12VA
- C4 pad 1: +VA -> +12VA
- C5 pad 1: +VA -> +12VA
- C6 pad 1: +VB -> +12VA
- C7 pad 1: +VB -> +12VA
- C8 pad 1: +VC -> +12VA
- C9 pad 1: +VC -> +12VA
- U4 pad 6: +VA -> +12VA
- U5 pad 6: +VB -> +12VA
- U6 pad 6: +VC -> +12VA
- U7 pad 6: +VD -> +12VA
Routing:
- net +12VA: track 24.4 -> 201.6 mm, vias 0 -> 2
- net +VA: track 68.5 -> 40.2 mm
- net +VB: track 68.0 -> 40.2 mm
- net +VC: track 65.1 -> 38.7 mm
- net +VD: track 66.1 -> 40.2 mm
- net GNDREF: track 506.5 -> 510.3 mm, vias 6 -> 10
- net Net-(D3-Pad2): track 14.9 -> 17.3 mm
- net Net-(R5-Pad2): track 9.51 -> 8.07 mm
Other:
- board text added: "VDC 1/2"
- board text added: "VDC 3/4"
- board text added: "VDC 5/6"
- board text added: "VDC 7/8"
- board text removed: "12VDC 1/2"
- board text removed: "12VDC 3/4"
- board text removed: "12VDC 5/6"
- board text removed: "12VDC 7/8"

Commit message: Update ESP-pwm-8ch-V1.kicad_pcb
Other:
- board text added: "8x PWM OUT 12/24VDC"
- board text removed: "8x PWM OUT 12VDC"
Changed lines of the file:
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@@
     (effects (font (size 1.5 1) (thickness 0.25)))
   )
-  (gr_text "8x PWM OUT 12VDC" (at 95.25 127) (layer "F.SilkS")
+  (gr_text "8x PWM OUT 12/24VDC" (at 95.25 127) (layer "F.SilkS")
     (effects (font (size 1.8 1.5) (thickness 0.25)))
   )

Commit message: Update ESP-pwm-8ch-V1.kicad_pcb
Parts:
- removed G***: LOGO, Tales:TMaschio_20mm
Other:
- board text added: "TMASCHIO 2022"

Commit message: updated connectors
Parts:
- removed REF**: OSHW-Logo2_14.6x12mm_SilkScreen, Symbol:OSHW-Logo2_14.6x12mm_SilkScreen
